File: hardware/wAveC/rev_a/wAveC.brd (EAGLE design)
At the start: 85.7 x 34.9 mm, 4 parts, among them J1 WIRE_HOLE-14AWG, J2 WIRE_HOLE-14AWG

Commit message: wavec routed
Parts:
- added J3, J4: MOLEX_BNC_73100-0105, connector:MOLEX-BNC-73100-0105
- moved J1 3.81 mm to (63.5, 28.6)
- turned R1 to 180 degrees
Connections:
- net CURRENT: now also J3.SIGNAL
- net GND: now also J3.GND1, J3.GND2
- net PHASE: now also J4.SIGNAL
Routing:
- net PHASE: track 0.00 -> 15.4 mm
- added copper zone on layer 1, net CURRENT
- added copper zone on layer 1, net GND
- added copper zone on layer 1, net PHASE
- added copper zone on layer 16, net PHASE
Changed lines of the file:
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@@
 <layer number="43" name="vRestrict" color="2" fill="10" visible="yes" active="yes"/>
 <layer number="44" name="Drills" color="7" fill="1" visible="no" active="yes"/>
-<layer number="45" name="Holes" color="7" fill="1" visible="no" active="yes"/>
+<layer number="45" name="Holes" color="7" fill="1" visible="yes" active="yes"/>
 <layer number="46" name="Milling" color="3" fill="1" visible="no" active="yes"/>
 <layer number="47" name="Measures" color="7" fill="1" visible="no" active="yes"/>
@@
 <wire x1="82.55" y1="25.4" x2="85.725" y2="25.4" width="0" layer="20"/>
 <wire x1="85.725" y1="25.4" x2="85.725" y2="9.525" width="0" layer="20"/>
+<wire x1="42.8625" y1="50.8" x2="42.8625" y2="-12.7" width="0.4064" layer="51"/>
+<hole x="2.8956" y="12.7" drill="3.175"/>
+<circle x="2.8956" y="12.7" radius="2.8448" width="0.4064" layer="51"/>
+<hole x="2.8956" y="22.225" drill="3.175"/>
+<circle x="2.8956" y="22.225" radius="2.8448" width="0.4064" layer="51"/>
+<hole x="82.8294" y="12.7" drill="3.175"/>
+<circle x="82.8294" y="12.7" radius="2.8448" width="0.4064" layer="51"/>
+<hole x="82.8294" y="22.225" drill="3.175"/>
+<circle x="82.8294" y="22.225" radius="2.8448" width="0.4064" layer="51"/>
 </plain>
 <attributes>
@@
 </autorouter>
 <elements>
-<element name="CT1" library="ac" package="CR8348" value="CR8348-1000" x="41.5925" y="12.065" rot="R90">
+<element name="CT1" library="ac" package="CR8348" value="CR8348-1000" x="41.5925" y="12.065" smashed="yes" rot="R90">
 <attribute name="DIGIKEY" value="582-1161-ND" x="47.9425" y="37.465" size="1.778" layer="27" rot="R90" display="off"/>
+<attribute name="NAME" x="41.275" y="24.0975" size="1.016" layer="21" font="vector" ratio="12" align="bottom-center"/>
 </element>
-<element name="R1" library="rcl" package="R1210" value="160" x="32.385" y="12.065" rot="R270">
-<attribute name="DIGIKEY" value="P160QCT-ND" x="32.385" y="12.065" size="1.778" layer="27" rot="R270" display="off"/>
+<element name="R1" library="rcl" package="R1210" value="160" x="32.385" y="12.065" smashed="yes" rot="R180">
+<attribute name="DIGIKEY" value="P160QCT-ND" x="32.385" y="12.065" size="1.778" layer="27" rot="R180" display="off"/>
+<attribute name="NAME" x="32.385" y="10.16" size="1.016" layer="25" font="vector" ratio="12" rot="R180" align="bottom-center"/>
+<attribute name="VALUE" x="34.925" y="15.24" size="1.27" layer="27" rot="R180"/>
 </element>
-<element name="J1" library="ac" package="WIRE_HOLE-14AWG" value="WIRE_HOLE-14AWG" x="59.69" y="28.575"/>
-<element name="J2" library="ac" package="WIRE_HOLE-14AWG" value="WIRE_HOLE-14AWG" x="70.485" y="28.575"/>
+<element name="J1" library="ac" package="WIRE_HOLE-14AWG" value="WIRE_HOLE-14AWG" x="63.5" y="28.575" smashed="yes"/>
+<element name="J2" library="ac" package="WIRE_HOLE-14AWG" value="WIRE_HOLE-14AWG" x="70.485" y="28.575" smashed="yes"/>
+<element name="J3" library="connector" package="MOLEX-BNC-73100-0105" value="MOLEX_BNC_73100-0105" x="33.02" y="26.416" smashed="yes" rot="R180">
+<attribute name="DIGIKEY" value="WM5524-ND" x="33.02" y="26.416" size="1.778" layer="27" rot="R180" display="off"/>
+<attribute name="NAME" x="29.21" y="25.861" size="1.016" layer="25" font="vector" ratio="12" rot="R180" align="bottom-center"/>
+</element>
+<element name="J4" library="connector" package="MOLEX-BNC-73100-0105" value="MOLEX_BNC_73100-0105" x="52.705" y="26.416" smashed="yes" rot="R180">
+<attribute name="DIGIKEY" value="WM5524-ND" x="52.705" y="26.416" size="1.778" layer="27" rot="R180" display="off"/>
+<attribute name="NAME" x="48.26" y="25.861" size="1.016" layer="25" font="vector" ratio="12" rot="R180" align="bottom-center"/>
+</element>
 </elements>
 <signals>
@@
 <contactref element="CT1" pad="1"/>
 <contactref element="R1" pad="2"/>
-<wire x1="32.385" y1="10.665" x2="36.8425" y2="4.465" width="0" layer="19" extent="1-1"/>
+<contactref element="J3" pad="SIGNAL"/>
+<polygon width="0.254" layer="1" thermals="no">
+<vertex x="31.75" y="22.86"/>
+<vertex x="29.21" y="13.97"/>
+<vertex x="29.21" y="10.16"/>
+<vertex x="35.56" y="3.175"/>
+<vertex x="38.1" y="3.175"/>
+<vertex x="38.1" y="6.35"/>
+<vertex x="35.56" y="6.35"/>
+<vertex x="31.75" y="10.795"/>
+<vertex x="31.75" y="13.97"/>
+<vertex x="34.29" y="22.225"/>
+<vertex x="34.29" y="23.495"/>
+<vertex x="31.75" y="23.495"/>
+</polygon>
 </signal>
 <signal name="GND">
 <contactref element="CT1" pad="2"/>
 <contactref element="R1" pad="1"/>
-<wire x1="32.385" y1="13.465" x2="36.8425" y2="19.665" width="0" layer="19" extent="1-1"/>
+<contactref element="J3" pad="GND1"/>
+<contactref element="J3" pad="GND2"/>
+<polygon width="0.254" layer="1" thermals="no">
+<vertex x="27.94" y="31.75"/>
+<vertex x="27.94" y="29.21"/>
+<vertex x="35.56" y="29.21"/>
+<vertex x="35.56" y="19.05"/>
+<vertex x="33.02" y="13.97"/>
+<vertex x="33.02" y="10.795"/>
+<vertex x="34.925" y="10.795"/>
+<vertex x="34.925" y="13.97"/>
+<vertex x="38.1" y="19.685"/>
+<vertex x="38.1" y="31.75"/>
+</polygon>
 </signal>
 <signal name="PHASE">
 <contactref element="J2" pad="P$1"/>
 <contactref element="J1" pad="P$1"/>
-<wire x1="59.69" y1="28.575" x2="70.485" y2="28.575" width="0" layer="19" extent="1-1"/>
+<contactref element="J4" pad="SIGNAL"/>
+<polygon width="0.4064" layer="1" thermals="no">
+<vertex x="60.325" y="31.75"/>
+<vertex x="60.325" y="25.4"/>
+<vertex x="73.025" y="25.4"/>
+<vertex x="73.025" y="31.75"/>
+</polygon>
+<polygon width="0.4064" layer="16" thermals="no">
+<vertex x="60.325" y="31.75"/>
+<vertex x="60.325" y="25.4"/>
+<vertex x="73.025" y="25.4"/>
+<vertex x="73.025" y="31.75"/>
+</polygon>
+<wire x1="63.5" y1="28.575" x2="63.5" y2="25.4" width="0.8128" layer="1"/>
+<wire x1="63.5" y1="25.4" x2="60.325" y2="22.225" width="0.8128" layer="1"/>
+<wire x1="60.325" y1="22.225" x2="52.996" y2="22.225" width="0.8128" layer="1"/>
+<wire x1="52.996" y1="22.225" x2="52.705" y2="22.516" width="0.8128" layer="1"/>
 </signal>
 </signals>

Commit message: added silkscreen
Parts:
- added LOGO1: UMICH_SOLID_MEDIUM, logos:UMICH_SOLID_200MIL
Other:
- board text added: "2014/05/19"
- board text added: "A"
- board text added: "Brad Campbell"
- board text added: "Current"
- board text added: "Phase"
- board text added: "Voltage"
- board text added: "wAveC"
Changed lines of the file:
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@@
 <layer number="20" name="Dimension" color="15" fill="1" visible="yes" active="yes"/>
 <layer number="21" name="tPlace" color="7" fill="1" visible="yes" active="yes"/>
-<layer number="22" name="bPlace" color="7" fill="1" visible="yes" active="yes"/>
+<layer number="22" name="bPlace" color="7" fill="1" visible="no" active="yes"/>
 <layer number="23" name="tOrigins" color="15" fill="1" visible="yes" active="yes"/>
-<layer number="24" name="bOrigins" color="15" fill="1" visible="yes" active="yes"/>
+<layer number="24" name="bOrigins" color="15" fill="1" visible="no" active="yes"/>
 <layer number="25" name="tNames" color="7" fill="1" visible="yes" active="yes"/>
-<layer number="26" name="bNames" color="7" fill="1" visible="yes" active="yes"/>
-<layer number="27" name="tValues" color="7" fill="1" visible="yes" active="yes"/>
-<layer number="28" name="bValues" color="7" fill="1" visible="yes" active="yes"/>
+<layer number="26" name="bNames" color="7" fill="1" visible="no" active="yes"/>
+<layer number="27" name="tValues" color="7" fill="1" visible="no" active="yes"/>
+<layer number="28" name="bValues" color="7" fill="1" visible="no" active="yes"/>
 <layer number="29" name="tStop" color="7" fill="3" visible="no" active="yes"/>
 <layer number="30" name="bStop" color="7" fill="6" visible="no" active="yes"/>
@@
 <wire x1="85.725" y1="25.4" x2="85.725" y2="9.525" width="0" layer="20"/>
 <wire x1="42.8625" y1="50.8" x2="42.8625" y2="-12.7" width="0.4064" layer="51"/>
-<hole x="2.8956" y="12.7" drill="3.175"/>
-<circle x="2.8956" y="12.7" radius="2.8448" width="0.4064" layer="51"/>
-<hole x="2.8956" y="22.225" drill="3.175"/>
-<circle x="2.8956" y="22.225" radius="2.8448" width="0.4064" layer="51"/>
-<hole x="82.8294" y="12.7" drill="3.175"/>
-<circle x="82.8294" y="12.7" radius="2.8448" width="0.4064" layer="51"/>
-<hole x="82.8294" y="22.225" drill="3.175"/>
-<circle x="82.8294" y="22.225" radius="2.8448" width="0.4064" layer="51"/>
+<hole x="3.175" y="12.7" drill="3.175"/>
+<circle x="3.175" y="12.7" radius="2.8448" width="0.4064" layer="51"/>
+<hole x="3.175" y="22.225" drill="3.175"/>
+<circle x="3.175" y="22.225" radius="2.8448" width="0.4064" layer="51"/>
+<hole x="82.55" y="12.7" drill="3.175"/>
+<circle x="82.55" y="12.7" radius="2.8448" width="0.4064" layer="51"/>
+<hole x="82.55" y="22.225" drill="3.175"/>
+<circle x="82.55" y="22.225" radius="2.8448" width="0.4064" layer="51"/>
+<text x="27.305" y="30.48" size="1.27" layer="21" font="vector" ratio="12" rot="R90" align="bottom-center">Current</text>
+<text x="46.99" y="30.48" size="1.27" layer="21" font="vector" ratio="12" rot="R90" align="bottom-center">Voltage</text>
+<text x="66.675" y="32.385" size="1.27" layer="21" font="vector" ratio="12" align="bottom-center">Phase</text>
+<text x="10.795" y="28.575" size="1.27" layer="21" font="vector" ratio="12">Brad Campbell</text>
+<text x="10.795" y="26.67" size="1.27" layer="21" font="vector" ratio="12">2014/05/19</text>
+<text x="10.795" y="30.48" size="1.778" layer="21" font="vector" ratio="15">wAveC</text>
+<text x="12.7" y="3.175" size="1.778" layer="21" font="vector" ratio="12" align="center">A</text>
+<wire x1="10.795" y1="5.08" x2="14.605" y2="5.08" width="0.254" layer="21"/>
+<wire x1="14.605" y1="5.08" x2="14.605" y2="1.27" width="0.254" layer="21"/>
+<wire x1="14.605" y1="1.27" x2="10.795" y2="1.27" width="0.254" layer="21"/>
+<wire x1="10.795" y1="1.27" x2="10.795" y2="5.08" width="0.254" layer="21"/>
 </plain>
 <attributes>
@@
 <attribute name="NAME" x="48.26" y="25.861" size="1.016" layer="25" font="vector" ratio="12" rot="R180" align="bottom-center"/>
 </element>
+<element name="LOGO1" library="logos" package="UMICH_SOLID_200MIL" value="UMICH_SOLID_MEDIUM" x="67.945" y="1.27"/>
 </elements>
 <signals>

Commit message: updated wavec labels and date
Parts:
- J1, J2: value WIRE_HOLE-14AWG -> MOLEX_BNC_73100-0105; device ac:WIRE_HOLE-14AWG -> connector:MOLEX-BNC-73100-0105
- J3, J4: value MOLEX_BNC_73100-0105 -> WIRE_HOLE-14AWG; device connector:MOLEX-BNC-73100-0105 -> ac:WIRE_HOLE-14AWG
- moved J1 30.6 mm to (33.0, 26.4), turned to 180 degrees
- moved J3 30.6 mm to (63.5, 28.6), turned to 0 degrees
- moved J2 17.9 mm to (52.7, 26.4), turned to 180 degrees
- moved J4 17.9 mm to (70.5, 28.6), turned to 0 degrees
Connections:
- net CURRENT: now also J1.SIGNAL; no longer J3.SIGNAL
- net GND: now also J1.GND1, J1.GND2; no longer J3.GND1, J3.GND2
- net PHASE: now also J2.SIGNAL, J3.P$1, J4.P$1; no longer J1.P$1, J2.P$1, J4.SIGNAL
Other:
- board text added: "2014/06/08"
- board text added: "Phase (BLK)"
- board text removed: "2014/05/19"
- board text removed: "Phase"
Changed lines of the file:
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@@
 <setting verticaltext="up"/>
 </settings>
-<grid distance="0.125" unitdist="inch" unit="inch" style="lines" multiple="1" display="yes" altdistance="0.025" altunitdist="inch" altunit="inch"/>
+<grid distance="0.0625" unitdist="inch" unit="inch" style="lines" multiple="1" display="yes" altdistance="0.025" altunitdist="inch" altunit="inch"/>
 <layers>
 <layer number="1" name="Top" color="4" fill="1" visible="yes" active="yes"/>
@@
 <text x="27.305" y="30.48" size="1.27" layer="21" font="vector" ratio="12" rot="R90" align="bottom-center">Current</text>
 <text x="46.99" y="30.48" size="1.27" layer="21" font="vector" ratio="12" rot="R90" align="bottom-center">Voltage</text>
-<text x="66.675" y="32.385" size="1.27" layer="21" font="vector" ratio="12" align="bottom-center">Phase</text>
+<text x="66.675" y="32.385" size="1.27" layer="21" font="vector" ratio="12" align="bottom-center">Phase (BLK)</text>
 <text x="10.795" y="28.575" size="1.27" layer="21" font="vector" ratio="12">Brad Campbell</text>
-<text x="10.795" y="26.67" size="1.27" layer="21" font="vector" ratio="12">2014/05/19</text>
+<text x="10.795" y="26.67" size="1.27" layer="21" font="vector" ratio="12">2014/06/08</text>
 <text x="10.795" y="30.48" size="1.778" layer="21" font="vector" ratio="15">wAveC</text>
 <text x="12.7" y="3.175" size="1.778" layer="21" font="vector" ratio="12" align="center">A</text>
@@
 <attribute name="VALUE" x="34.925" y="15.24" size="1.27" layer="27" rot="R180"/>
 </element>
-<element name="J1" library="ac" package="WIRE_HOLE-14AWG" value="WIRE_HOLE-14AWG" x="63.5" y="28.575" smashed="yes"/>
-<element name="J2" library="ac" package="WIRE_HOLE-14AWG" value="WIRE_HOLE-14AWG" x="70.485" y="28.575" smashed="yes"/>
-<element name="J3" library="connector" package="MOLEX-BNC-73100-0105" value="MOLEX_BNC_73100-0105" x="33.02" y="26.416" smashed="yes" rot="R180">
+<element name="J3" library="ac" package="WIRE_HOLE-14AWG" value="WIRE_HOLE-14AWG" x="63.5" y="28.575" smashed="yes"/>
+<element name="J4" library="ac" package="WIRE_HOLE-14AWG" value="WIRE_HOLE-14AWG" x="70.485" y="28.575" smashed="yes"/>
+<element name="J1" library="connector" package="MOLEX-BNC-73100-0105" value="MOLEX_BNC_73100-0105" x="33.02" y="26.416" smashed="yes" rot="R180">
 <attribute name="DIGIKEY" value="WM5524-ND" x="33.02" y="26.416" size="1.778" layer="27" rot="R180" display="off"/>
 <attribute name="NAME" x="29.21" y="25.861" size="1.016" layer="25" font="vector" ratio="12" rot="R180" align="bottom-center"/>
 </element>
-<element name="J4" library="connector" package="MOLEX-BNC-73100-0105" value="MOLEX_BNC_73100-0105" x="52.705" y="26.416" smashed="yes" rot="R180">
+<element name="J2" library="connector" package="MOLEX-BNC-73100-0105" value="MOLEX_BNC_73100-0105" x="52.705" y="26.416" smashed="yes" rot="R180">
 <attribute name="DIGIKEY" value="WM5524-ND" x="52.705" y="26.416" size="1.778" layer="27" rot="R180" display="off"/>
 <attribute name="NAME" x="48.26" y="25.861" size="1.016" layer="25" font="vector" ratio="12" rot="R180" align="bottom-center"/>
@@
 <contactref element="CT1" pad="1"/>
 <contactref element="R1" pad="2"/>
-<contactref element="J3" pad="SIGNAL"/>
+<contactref element="J1" pad="SIGNAL"/>
 <polygon width="0.254" layer="1" thermals="no">
 <vertex x="31.75" y="22.86"/>
@@
 <contactref element="CT1" pad="2"/>
 <contactref element="R1" pad="1"/>
-<contactref element="J3" pad="GND1"/>
-<contactref element="J3" pad="GND2"/>
+<contactref element="J1" pad="GND1"/>
+<contactref element="J1" pad="GND2"/>
 <polygon width="0.254" layer="1" thermals="no">
 <vertex x="27.94" y="31.75"/>
@@
 </signal>
 <signal name="PHASE">
-<contactref element="J2" pad="P$1"/>
-<contactref element="J1" pad="P$1"/>
-<contactref element="J4" pad="SIGNAL"/>
+<contactref element="J4" pad="P$1"/>
+<contactref element="J3" pad="P$1"/>
+<contactref element="J2" pad="SIGNAL"/>
 <polygon width="0.4064" layer="1" thermals="no">
 <vertex x="60.325" y="31.75"/>
